Commit message: Added code to build hexapod based on the loaded urdf model. Added 22 leg example urdf. Updated all urdfs in line with new naming convention.

File: vis/urdf/hexapod.urdf.xacro (robot description, xacro)
@@ -4,5 +4,5 @@
   <xacro:property name="length" value="1.8" />
   <xacro:property name="width" value="1.0" />
-  <xacro:property name="depth" value="0.2" />
+  <xacro:property name="depth" value="${width/5.0}" />
   <xacro:property name="joint_1_lower_limit" value="${-pi}" />
   <xacro:property name="joint_1_upper_limit" value="${pi}" />
@@ -33,14 +33,8 @@
   </xacro:macro >
   <xacro:macro name="leg" params="position side reflect_leftright reflect_frontback">
-  <joint name="base_to_leg_${position}_${side}_link_0" type="fixed">
+  <joint name="leg_${position}_${side}_joint_1" type="revolute">
     <parent link="body_link"/>
-    <child link="leg_${position}_${side}_link_0"/>
+    <child link="leg_${position}_${side}_link_1"/>
     <origin rpy="0 0 ${reflect_leftright*pi/2}" xyz="${reflect_frontback*(length/2)*0.6666666} ${reflect_leftright*width/2} 0"/>
-  </joint>
-  <link name="leg_${position}_${side}_link_0">
-  </link>
-  <joint name="leg_${position}_${side}_joint_1" type="revolute">
-    <parent link="leg_${position}_${side}_link_0"/>
-    <child link="leg_${position}_${side}_link_1"/>
     <axis xyz="0 0 1"/>
     <limit lower="${joint_1_lower_limit}" upper="${joint_1_upper_limit}" effort="100" velocity="100" />
@@ -121,9 +115,9 @@
   </link>
   </xacro:macro>
-  <xacro:leg position="front" side="left" reflect_leftright="1" reflect_frontback="1"/>
-  <xacro:leg position="mid1" side="left" reflect_leftright="1" reflect_frontback="0"/>
-  <xacro:leg position="back" side="left" reflect_leftright="1" reflect_frontback="-1"/>
-  <xacro:leg position="front" side="right" reflect_leftright="-1" reflect_frontback="1"/>
-  <xacro:leg position="mid1" side="right" reflect_leftright="-1" reflect_frontback="0"/>
-  <xacro:leg position="back" side="right" reflect_leftright="-1" reflect_frontback="-1"/>
+  <xacro:leg position="row00" side="left" reflect_leftright="1" reflect_frontback="1"/>
+  <xacro:leg position="row00" side="right" reflect_leftright="-1" reflect_frontback="1"/>
+  <xacro:leg position="row01" side="left" reflect_leftright="1" reflect_frontback="0"/>
+  <xacro:leg position="row01" side="right" reflect_leftright="-1" reflect_frontback="0"/>
+  <xacro:leg position="row02" side="left" reflect_leftright="1" reflect_frontback="-1"/>
+  <xacro:leg position="row02" side="right" reflect_leftright="-1" reflect_frontback="-1"/>
 </robot>

File: vis/urdf/hexapod2.urdf.xacro (robot description, xacro)
@@ -4,5 +4,5 @@
   <xacro:property name="length" value="1.8" />
   <xacro:property name="width" value="1.0" />
-  <xacro:property name="depth" value="0.2" />
+  <xacro:property name="depth" value="${width/5.0}" />
   <xacro:property name="joint_1_lower_limit" value="${-pi}" />
   <xacro:property name="joint_1_upper_limit" value="${pi}" />
@@ -33,14 +33,8 @@
   </xacro:macro >
   <xacro:macro name="leg" params="position side reflect_leftright reflect_frontback">
-  <joint name="base_to_leg_${position}_${side}_link_0" type="fixed">
+  <joint name="leg_${position}_${side}_joint_1" type="revolute">
     <parent link="body_link"/>
-    <child link="leg_${position}_${side}_link_0"/>
+    <child link="leg_${position}_${side}_link_1"/>
     <origin rpy="0 0 ${reflect_leftright*(pi/2 - reflect_frontback*pi/6)}" xyz="${reflect_frontback*(length/2)} ${reflect_leftright*width/2} 0"/>
-  </joint>
-  <link name="leg_${position}_${side}_link_0">
-  </link>
-  <joint name="leg_${position}_${side}_joint_1" type="revolute">
-    <parent link="leg_${position}_${side}_link_0"/>
-    <child link="leg_${position}_${side}_link_1"/>
     <axis xyz="0 0 1"/>
     <limit lower="${joint_1_lower_limit}" upper="${joint_1_upper_limit}" effort="100" velocity="100" />
@@ -121,9 +115,9 @@
   </link>
   </xacro:macro>
-  <xacro:leg position="front" side="left" reflect_leftright="1" reflect_frontback="1"/>
-  <xacro:leg position="mid1" side="left" reflect_leftright="1" reflect_frontback="0"/>
-  <xacro:leg position="back" side="left" reflect_leftright="1" reflect_frontback="-1"/>
-  <xacro:leg position="front" side="right" reflect_leftright="-1" reflect_frontback="1"/>
-  <xacro:leg position="mid1" side="right" reflect_leftright="-1" reflect_frontback="0"/>
-  <xacro:leg position="back" side="right" reflect_leftright="-1" reflect_frontback="-1"/>
+  <xacro:leg position="row00" side="left" reflect_leftright="1" reflect_frontback="1"/>
+  <xacro:leg position="row00" side="right" reflect_leftright="-1" reflect_frontback="1"/>
+  <xacro:leg position="row01" side="left" reflect_leftright="1" reflect_frontback="0"/>
+  <xacro:leg position="row01" side="right" reflect_leftright="-1" reflect_frontback="0"/>
+  <xacro:leg position="row02" side="left" reflect_leftright="1" reflect_frontback="-1"/>
+  <xacro:leg position="row02" side="right" reflect_leftright="-1" reflect_frontback="-1"/>
 </robot>

File: vis/urdf/sillypod.urdf.xacro (robot description, xacro)
@@ -2,5 +2,5 @@
 <robot name="hexapod" xmlns:xacro="http://ros.org/wiki/xacro">
   <xacro:property name="pi" value="3.1415926535897931" />
-  <xacro:property name="length" value="1.8" />
+  <xacro:property name="length" value="10.0" />
   <xacro:property name="width" value="1.0" />
   <xacro:property name="depth" value="${width/5.0}" />
@@ -116,11 +116,25 @@
   </link>
   </xacro:macro>
-  <xacro:leg position="row00" side="left" reflect_leftright="1" forward_position="${length/2}" />
-  <xacro:leg position="row01" side="left" reflect_leftright="1" forward_position="${length/2 - (length/(num_legs/2-1))}" />
-  <xacro:leg position="row02" side="left" reflect_leftright="1" forward_position="${-length/2 + (length/(num_legs/2-1))}" />
-  <xacro:leg position="row03" side="left" reflect_leftright="1" forward_position="${-length/2}" />
-  <xacro:leg position="row00" side="right" reflect_leftright="-1" forward_position="${length/2}" />
-  <xacro:leg position="row01" side="right" reflect_leftright="-1" forward_position="${length/2 - (length/(num_legs/2-1))}" />
-  <xacro:leg position="row02" side="right" reflect_leftright="-1" forward_position="${-length/2 + (length/(num_legs/2-1))}" />
-  <xacro:leg position="row03" side="right" reflect_leftright="-1" forward_position="${-length/2}" />
+  <xacro:leg position="row00" side="left" reflect_leftright="1" forward_position="5" />
+  <xacro:leg position="row01" side="left" reflect_leftright="1" forward_position="4" />
+  <xacro:leg position="row02" side="left" reflect_leftright="1" forward_position="3" />
+  <xacro:leg position="row03" side="left" reflect_leftright="1" forward_position="2" />
+  <xacro:leg position="row04" side="left" reflect_leftright="1" forward_position="1" />
+  <xacro:leg position="row05" side="left" reflect_leftright="1" forward_position="0" />
+  <xacro:leg position="row06" side="left" reflect_leftright="1" forward_position="-1" />
+  <xacro:leg position="row07" side="left" reflect_leftright="1" forward_position="-2" />
+  <xacro:leg position="row08" side="left" reflect_leftright="1" forward_position="-3" />
+  <xacro:leg position="row09" side="left" reflect_leftright="1" forward_position="-4" />
+  <xacro:leg position="row10" side="left" reflect_leftright="1" forward_position="-5" />
+  <xacro:leg position="row00" side="right" reflect_leftright="-1" forward_position="5" />
+  <xacro:leg position="row01" side="right" reflect_leftright="-1" forward_position="4" />
+  <xacro:leg position="row02" side="right" reflect_leftright="-1" forward_position="3" />
+  <xacro:leg position="row03" side="right" reflect_leftright="-1" forward_position="2" />
+  <xacro:leg position="row04" side="right" reflect_leftright="-1" forward_position="1" />
+  <xacro:leg position="row05" side="right" reflect_leftright="-1" forward_position="0" />
+  <xacro:leg position="row06" side="right" reflect_leftright="-1" forward_position="-1" />
+  <xacro:leg position="row07" side="right" reflect_leftright="-1" forward_position="-2" />
+  <xacro:leg position="row08" side="right" reflect_leftright="-1" forward_position="-3" />
+  <xacro:leg position="row09" side="right" reflect_leftright="-1" forward_position="-4" />
+  <xacro:leg position="row10" side="right" reflect_leftright="-1" forward_position="-5" />
 </robot>

Commit message: Remove redeclared xacro variable (pi).

File: vis/urdf/hexapod.urdf.xacro (robot description, xacro)
@@ -1,5 +1,4 @@
 <?xml version="1.0"?>
 <robot name="hexapod" xmlns:xacro="http://ros.org/wiki/xacro">
-  <xacro:property name="pi" value="3.1415926535897931" />
   <xacro:property name="length" value="1.8" />
   <xacro:property name="width" value="1.0" />

File: vis/urdf/hexapod2.urdf.xacro (robot description, xacro)
@@ -1,5 +1,4 @@
 <?xml version="1.0"?>
 <robot name="hexapod" xmlns:xacro="http://ros.org/wiki/xacro">
-  <xacro:property name="pi" value="3.1415926535897931" />
   <xacro:property name="length" value="1.8" />
   <xacro:property name="width" value="1.0" />

File: vis/urdf/octapod.urdf.xacro (robot description, xacro)
@@ -1,5 +1,4 @@
 <?xml version="1.0"?>
 <robot name="hexapod" xmlns:xacro="http://ros.org/wiki/xacro">
-  <xacro:property name="pi" value="3.1415926535897931" />
   <xacro:property name="length" value="1.8" />
   <xacro:property name="width" value="1.0" />

File: vis/urdf/sillypod.urdf.xacro (robot description, xacro)
@@ -1,5 +1,4 @@
 <?xml version="1.0"?>
 <robot name="hexapod" xmlns:xacro="http://ros.org/wiki/xacro">
-  <xacro:property name="pi" value="3.1415926535897931" />
   <xacro:property name="length" value="10.0" />
   <xacro:property name="width" value="1.0" />
