Commit message: Correct joint3 offset (was previously given wrt non-offset joint 2).

File: vis/urdf/phantomx.urdf.xacro (robot description, xacro)
@@ -13,4 +13,5 @@
   <xacro:property name="tibia_length" value="0.132" />
   <!-- Rough limits. Offsets from manual measurements again. -->
+  <!-- TODO update limits. -->
   <xacro:property name="joint_1_lower_limit" value="${-pi}" />
   <xacro:property name="joint_1_upper_limit" value="${pi}" />
@@ -88,5 +89,5 @@
     <parent link="leg_${row}_${side}_link_2"/>
     <child link="leg_${row}_${side}_link_3"/>
-    <origin rpy="0 0 -${joint_3_offset}" xyz="${femur_length} 0 0"/>
+    <origin rpy="0 0 ${-(joint_3_offset-joint_2_offset)}" xyz="${femur_length} 0 0"/>
     <axis xyz="0 0 1"/>
     <limit lower="${joint_3_lower_limit}" upper="${joint_3_upper_limit}" effort="100" velocity="100" />

Commit message: Fix joint 3 offset in phantom x urdf

File: vis/urdf/phantomx.urdf.xacro (robot description, xacro)
@@ -21,5 +21,5 @@
   <xacro:property name="joint_3_lower_limit" value="${-pi}" />
   <xacro:property name="joint_3_upper_limit" value="${pi}" />
-  <xacro:property name="joint_3_offset" value="${46.0*pi/180.0}" />
+  <xacro:property name="joint_3_offset" value="${32.0*pi/180.0}" />
   <link name="base_link">
   </link>
